File: Schematics/CNTRL/CNTRL.kicad_pcb (KiCad board)
At the start: 4 copper layers, 78 x 78 mm, 132 parts, among them J1 SWD, J10 Y+, J11 Y-, J12 693071020811, J13 3.3V, J14 NAVIG I2C, J15 I2C, J16 USART, J17 PYRO1_OSTTE020104, J18 PYRO3_OSTTE020104, J19 USB_A_TE_292303-7_Horizontal, J2 CONSMA001-SMD-G-T, J20 PYRO2_OSTTE020104, J21 PYRO4_OSTTE020104, J3 3S LiPo, J4 F4, J5 F3, J6 F2, J7 F1, J8 X+, J9 X-, Q1 BUK9832-55A_CUX, Q2 BUK9832-55A_CUX, Q3 BUK9832-55A_CUX, Q4 BUK9832-55A_CUX, Q5 BUK9832-55A_CUX, SW1 Omron_B3F-10xx, SW2 Omron_B3F-10xx, U1 STM32405RGT6, U10 TLP293GB-TPL_E, U11 TLP293GB-TPL_E, U2 RFM95W-915S2, U3 TPS2117DRLR, U4 TPS563200, U5 AMS1117-3.3, U6 TLP293GB-TPL_E, U7 W25Q128JVSIQ, U8 USBLC6-2SC6, U9 TLP293GB-TPL_E, Y1 12MHz_ECS-120-18-33-JGN-TR3, Y2 32.768KHz_SC32S-7PF20PPM

Commit message: CNTRL fixes towards v1.1
Parts:
- removed R28: 68, Resistor_SMD:R_0603_1608Metric
- removed R36: 10K, Resistor_SMD:R_0603_1608Metric
- removed U10, U11, U6, U9: TLP293GB-TPL_E, External:SO4_TOS
- added J22: Reset Jumper, Connector_PinHeader_2.54mm:PinHeader_1x02_P2.54mm_Vertical, F.Cu at (89.2, 96.8)
- added R45: 10K, Resistor_SMD:R_0603_1608Metric, F.Cu at (27.2, 79.5)
- added R46: 3.7K, Resistor_SMD:R_0603_1608Metric, F.Cu at (27.2, 82.0)
- R34: value 82K -> 10K
- R35: value 33K -> 4.7K
- R37, R41, R43: value 68 -> 10K
- R40, R42, R44: value 10K -> 3.7K
- Y2: value 32.768KHz_SC32S-7PF20PPM -> 32.768KHz_SC32S-7PF20PPM
- moved R43 29.3 mm to (27.2, 74.5)
- moved R44 29.3 mm to (27.2, 77.0)
- moved R42 29.3 mm to (27.2, 72.0)
- moved R37 25.4 mm to (27.2, 64.4)
- moved R40 25.4 mm to (27.2, 66.9)
- moved R41 25.4 mm to (27.2, 69.5)
- moved C3 6.25 mm to (93.0, 96.8)
Connections:
- R37 pad 1: Net-(R37-Pad1) -> Net-(Q3-Pad2)
- R37 pad 2: +3.3V -> PYRO_2_SENSE
- R40 pad 1: +3.3V -> PYRO_2_SENSE
- R40 pad 2: PYRO_2_SENSE -> GND
- R41 pad 1: Net-(R41-Pad1) -> Net-(Q2-Pad2)
- R41 pad 2: +3.3V -> PYRO_3_SENSE
- R42 pad 1: +3.3V -> PYRO_3_SENSE
- R42 pad 2: PYRO_4_SENSE -> GND
- R43 pad 1: Net-(R43-Pad1) -> Net-(Q4-Pad2)
- R43 pad 2: +3.3V -> PYRO_4_SENSE
- R44 pad 1: +3.3V -> PYRO_4_SENSE
- R44 pad 2: PYRO_3_SENSE -> GND
- SW2 pad 1: SWD_NRST -> Net-(J22-Pin_2)
Routing:
- net Net-(J22-Pin_2): track 0.00 -> 11.5 mm
- net SWD_NRST: track 103.9 -> 93.3 mm
Other:
- board text added: "v1.1"
- board text removed: "v1.0"

Commit message: CNTRL v1.1 fixes
Parts:
- removed J11: Y-, Connector_PinHeader_2.54mm:PinHeader_1x03_P2.54mm_Vertical
- removed J4: F4, Connector_PinHeader_2.54mm:PinHeader_1x03_P2.54mm_Vertical
- removed J7: F1, Connector_PinHeader_2.54mm:PinHeader_1x03_P2.54mm_Vertical
- removed J9: X-, Connector_PinHeader_2.54mm:PinHeader_1x03_P2.54mm_Vertical
- added C24: 100nF, Capacitor_SMD:C_0603_1608Metric, F.Cu at (146.8, 77.5)
- added C26: 100nF, Capacitor_SMD:C_0603_1608Metric, F.Cu at (149.0, 68.2)
- added C29: 470uF, Capacitor_THT:CP_Radial_D6.3mm_P2.50mm, F.Cu at (121.0, 118.0)
- added C30: 470uF, Capacitor_THT:CP_Radial_D6.3mm_P2.50mm, F.Cu at (129.2, 118.0)
- added C31: 100nF, Capacitor_SMD:C_0603_1608Metric, B.Cu at (120.5, 120.8)
- added C32: 100nF, Capacitor_SMD:C_0603_1608Metric, B.Cu at (129.8, 120.5)
- added J23: USB_C_Receptacle_USB2.0, Connector_USB:USB_C_Receptacle_GCT_USB4105-xx-A_16P_TopMnt_Horizontal, F.Cu at (127.2, 54.8)
- added J24: 5V, Connector_JST:JST_XH_B2B-XH-A_1x02_P2.50mm_Vertical, F.Cu at (91.0, 59.8)
- added R28: 10K, Resistor_SMD:R_0603_1608Metric, F.Cu at (145.2, 68.8)
- added R36: 5.1K, Resistor_SMD:R_0603_1608Metric, F.Cu at (128.5, 62.5)
- added R47: 5.1K, Resistor_SMD:R_0603_1608Metric, F.Cu at (124.8, 61.8)
- C23, C25, TP1, TP2, U5: moved to F.Cu
- J10: value Y+ -> Y; footprint Connector_PinHeader_2.54mm:PinHeader_1x03_P2.54mm_Vertical -> TerminalBlock_Phoenix:TerminalBlock_Phoenix_MPT-0,5-3-2.54_1x03_P2.54mm_Horizontal
- J15: value I2C -> ESP32 I2C
- J19: value USB_A_TE_292303-7_Horizontal -> 3.3V; footprint Connector_USB:USB_A_TE_292303-7_Horizontal -> Connector_JST:JST_XH_B2B-XH-A_1x02_P2.50mm_Vertical
- J5: value F3 -> GPIO 1-2; footprint Connector_PinHeader_2.54mm:PinHeader_1x03_P2.54mm_Vertical -> TerminalBlock_Phoenix:TerminalBlock_Phoenix_MPT-0,5-2-2.54_1x02_P2.54mm_Horizontal
- J6: value F2 -> GPIO 3-4; footprint Connector_PinHeader_2.54mm:PinHeader_1x03_P2.54mm_Vertical -> TerminalBlock_Phoenix:TerminalBlock_Phoenix_MPT-0,5-2-2.54_1x02_P2.54mm_Horizontal
- J8: value X+ -> X; footprint Connector_PinHeader_2.54mm:PinHeader_1x03_P2.54mm_Vertical -> TerminalBlock_Phoenix:TerminalBlock_Phoenix_MPT-0,5-3-2.54_1x03_P2.54mm_Horizontal
- Q1, Q2, Q3, Q4, Q5: footprint BUK9832-55A_CUX:TRANS_BUK9832-55A_CUX -> External:TRANS_BUK9832-55A_CUX
- R11, R22, R23, R43, R44: moved to B.Cu
- U7: footprint Package_SO:SOIC-8_5.23x5.23mm_P1.27mm -> Package_SO:SOIC-8_5.3x5.3mm_P1.27mm
- moved R43 121.1 mm to (145.0, 102.5), turned to 180 degrees
- moved R44 120.3 mm to (145.0, 101.0)
- moved R41 117.7 mm to (136.0, 114.2), turned to 180 degrees
- moved R42 116.2 mm to (136.0, 112.8)
- moved R11 91.2 mm to (135.8, 92.0)
- moved R23 89.5 mm to (135.8, 89.5)
- moved R37 86.4 mm to (97.8, 114.2)
- moved R40 84.1 mm to (97.8, 112.8), turned to 180 degrees
- moved R45 69.0 mm to (90.2, 107.5)
- moved R46 67.5 mm to (90.2, 106.0), turned to 180 degrees
- moved R22 64.9 mm to (106.8, 97.8), turned to 180 degrees
- moved R27 55.8 mm to (98.5, 99.0), turned to 180 degrees
- moved R1 45.9 mm to (87.0, 89.5), turned to -90 degrees
- moved J19 38.0 mm to (91.0, 71.5), turned to 45 degrees
- moved TP6 17.0 mm to (132.5, 61.2)
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Connections:
- C18 pad 1: VBUS -> BUCK_+5V
- J19 pad 1: VBUS -> +3.3V
- J19 pad 2: /USB_RAW_D- -> GND
- J5 pad 1: FIN_SERVO_3 -> IO1
- J5 pad 2: +5V -> IO2
- J6 pad 1: FIN_SERVO_2 -> IO3
- J6 pad 2: +5V -> IO4
- R4 pad 1: VBUS -> BUCK_+5V
- U1 pad 37: FIN_SERVO_1 -> IO1
- U1 pad 38: FIN_SERVO_2 -> IO2
- U1 pad 39: FIN_SERVO_3 -> IO3
- U1 pad 40: FIN_SERVO_4 -> IO4
- U3 pad 3: VBUS -> BUCK_+5V
- U3 pad 5: VBUS -> BUCK_+5V
- U3 pad 6: BUCK_+5V -> VBUS
- U4 pad 5: +BATT -> Net-(U4-EN)
Routing:
- net GND: track 14.0 -> 61.7 mm, vias 18 -> 26
- net +5V: track 175.9 -> 215.5 mm
- net FIN_SERVO_1: track 36.9 -> 0.00 mm
- net TVC_SERVO_Y: track 68.5 -> 33.0 mm
- net IO1: track 0.00 -> 34.7 mm
- net IO2: track 0.00 -> 33.8 mm
- net FIN_SERVO_2: track 33.6 -> 0.00 mm
- net IO3: track 0.00 -> 32.3 mm
- net IO4: track 0.00 -> 31.4 mm
- net FIN_SERVO_3: track 30.4 -> 0.00 mm
- net TVC_SERVO_X: track 57.8 -> 29.8 mm
- net FIN_SERVO_4: track 27.2 -> 0.00 mm
- net unconnected-(J19-Shield-Pad5): track 13.1 -> 0.00 mm
- net +3.3V: track 97.6 -> 107.1 mm, vias 16 -> 18
- net Net-(BZ1-+): track 10.9 -> 18.9 mm
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Other:
- board text added: "+"
- board text added: "-"
- board text added: "3.3V"
- board text added: "5V"
- board text added: "BEFORE FLIGHT!"
- board text added: "GPIO"
- board text added: "REMOVE JUMPER"
- board text added: "USART"
- board text added: "X"
- board text added: "Y"
- board text removed: "FINS"
- board text removed: "TVC"

Commit message: final CNTRL v1.1
Parts:
- added R48: 5K, Resistor_SMD:R_0603_1608Metric, F.Cu at (90.2, 106.0)
- added R49: 5K, Resistor_SMD:R_0603_1608Metric, F.Cu at (136.0, 112.8)
- added R50: 5K, Resistor_SMD:R_0603_1608Metric, B.Cu at (145.0, 101.0)
- added R51: 5K, Resistor_SMD:R_0603_1608Metric, F.Cu at (97.8, 112.8)
- R37, R41, R43, R45: value 10K -> 5K
- moved R44 1.53 mm to (145.0, 99.5)
- moved R40 1.50 mm to (97.8, 111.2)
- moved R42 1.50 mm to (136.0, 111.2)
- moved R46 1.50 mm to (90.2, 104.5)
Connections:
- R37 pad 2: PYRO_2_SENSE -> Net-(R37-Pad2)
- R41 pad 2: PYRO_3_SENSE -> Net-(R41-Pad2)
- R43 pad 2: PYRO_4_SENSE -> Net-(R43-Pad2)
- R45 pad 2: PYRO_1_SENSE -> Net-(R45-Pad2)
Routing:
- net PYRO_2_SENSE: track 43.7 -> 39.9 mm
- net GND: track 61.7 -> 59.4 mm, vias 26 -> 55
- net Net-(Q2-Pad2): track 15.4 -> 17.3 mm
- net Net-(R45-Pad2): track 0.00 -> 1.50 mm
- net Net-(R43-Pad2): track 0.00 -> 1.50 mm
- net Net-(R41-Pad2): track 0.00 -> 1.50 mm
- net Net-(R37-Pad2): track 0.00 -> 1.50 mm
- net PYRO_3_SENSE: track 45.1 -> 45.6 mm
Other:
- board text added: "Designed By: Arav Sonawane July 2025"
- board text removed: "Designed By: Arav Sonawane August 2024"

Commit message: CNTRL production run
Routing:
- net +3.3V: vias 18 -> 28
- added copper zone on F.Cu, net +3.3V
Changed lines of the file:
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@@
 	)
 	(segment
-		(start 141.475 75.25)
-		(end 141.5 75.225)
-		(width 0.5)
-		(layer "F.Cu")
-		(net 5)
-	)
-	(segment
 		(start 120.575 68.825)
 		(end 120.5 68.75)
@@
 	)
 	(segment
+		(start 138.9 75.25)
+		(end 141.475 75.25)
+		(width 1)
+		(layer "F.Cu")
+		(net 5)
+	)
+	(segment
 		(start 152 79)
 		(end 152.075 79.075)
@@
 	)
 	(segment
-		(start 138.9 75.25)
-		(end 141.475 75.25)
-		(width 0.5)
-		(layer "F.Cu")
-		(net 5)
-	)
-	(segment
 		(start 111.095 97.845)
 		(end 111.75 98.5)
@@
 	)
 	(segment
+		(start 141.475 75.25)
+		(end 141.5 75.225)
+		(width 1)
+		(layer "F.Cu")
+		(net 5)
+	)
+	(segment
 		(start 152.075 79.075)
 		(end 152.075 80.25)
@@
 	)
 	(via
+		(at 137 74.75)
+		(size 0.7)
+		(drill 0.3)
+		(layers "F.Cu" "B.Cu")
+		(net 5)
+	)
+	(via
+		(at 136 75.75)
+		(size 0.7)
+		(drill 0.3)
+		(layers "F.Cu" "B.Cu")
+		(net 5)
+	)
+	(via
 		(at 107 76)
 		(size 0.7)
@@
 	)
 	(via
+		(at 134.75 77.25)
+		(size 0.7)
+		(drill 0.3)
+		(layers "F.Cu" "B.Cu")
+		(net 5)
+	)
+	(via
 		(at 139 72)
 		(size 0.7)
@@
 	)
 	(via
+		(at 139 78.25)
+		(size 0.7)
+		(drill 0.3)
+		(layers "F.Cu" "B.Cu")
+		(net 5)
+	)
+	(via
+		(at 136 73.5)
+		(size 0.7)
+		(drill 0.3)
+		(layers "F.Cu" "B.Cu")
+		(net 5)
+	)
+	(via
+		(at 136 78.25)
+		(size 0.7)
+		(drill 0.3)
+		(layers "F.Cu" "B.Cu")
+		(net 5)
+	)
+	(via
 		(at 109.75 69)
 		(size 0.7)
@@
 	)
 	(via
+		(at 134.75 72.5)
+		(size 0.7)
+		(drill 0.3)
+		(layers "F.Cu" "B.Cu")
+		(net 5)
+	)
+	(via
 		(at 121.25 107.5)
 		(size 0.7)
@@
 	)
 	(via
+		(at 134.75 74.75)
+		(size 0.7)
+		(drill 0.3)
+		(layers "F.Cu" "B.Cu")
+		(net 5)
+	)
+	(via
 		(at 107.5 96.5)
 		(size 0.7)
@@
 		(net 5)
 	)
+	(via
+		(at 137 72.5)
+		(size 0.7)
+		(drill 0.3)
+		(layers "F.Cu" "B.Cu")
+		(net 5)
+	)
+	(via
+		(at 137 77.25)
+		(size 0.7)
+		(drill 0.3)
+		(layers "F.Cu" "B.Cu")
+		(net 5)
+	)
 	(segment
 		(start 117 66.925)
@@
 	)
 	(segment
-		(start 129.65 61.15)
-		(end 130 61.5)
-		(width 0.3)
-		(layer "F.Cu")
-		(net 10)
-	)
-	(segment
-		(start 126.751 69.501)
-		(end 127.261 69.501)
+		(start 124.85 59.8)
+		(end 124.85 58.43)
 		(width 0.3)
 		(layer "F.Cu")
@@
 	)
 	(segment
-		(start 121.5 64.25)
-		(end 126.751 69.501)
-		(width 0.3)
+		(start 121.5 61.25)
+		(end 122.25 60.5)
+		(width 0.5)
 		(layer "F.Cu")
 		(net 10)
 	)
 	(segment
-		(start 124.85 59.8)
-		(end 124.85 58.43)
-		(width 0.3)
+		(start 129.65 58.43)
+		(end 129.65 61.15)
+		(width 0.5)
 		(layer "F.Cu")
 		(net 10)
 	)
 	(segment
-		(start 129.65 58.43)
-		(end 129.65 61.15)
-		(width 0.3)
+		(start 124.15 60.5)
+		(end 124.75 59.9)
+		(width 0.5)
 		(layer "F.Cu")
 		(net 10)
@@
 	)
 	(segment
-		(start 121.5 61.25)
-		(end 121.5 64.25)
-		(width 0.3)
+		(start 126.001 69.501)
+		(end 121.5 65)
+		(width 0.5)
 		(layer "F.Cu")
 		(net 10)
 	)
 	(segment
-		(start 122.85 59.9)
+		(start 121.5 65)
 		(end 121.5 61.25)
-		(width 0.3)
+		(width 0.5)
 		(layer "F.Cu")
 		(net 10)
@@
 	)
 	(segment
-		(start 124.75 59.9)
-		(end 122.85 59.9)
-		(width 0.3)
+		(start 122.25 60.5)
+		(end 124.15 60.5)
+		(width 0.5)
 		(layer "F.Cu")
 		(net 10)
@@
 	)
 	(segment
+		(start 129.65 61.15)
+		(end 130 61.5)
+		(width 0.5)
+		(layer "F.Cu")
+		(net 10)
+	)
+	(segment
 		(start 125.750466 57)
 		(end 128.749534 57)
@@
 		(net 10)
 	)
+	(segment
+		(start 126.001 69.501)
+		(end 127.261 69.501)
+		(width 0.3)
+		(layer "F.Cu")
+		(net 10)
+	)
 	(via
 		(at 130 61.5)
@@
 			)
 		)
+	)
+	(zone
+		(net 5)
+		(net_name "+3.3V")
+		(layer "F.Cu")
+		(hatch edge 0.5)
+		(priority 4)
+		(connect_pads
+			(clearance 0.5)
+		)
+		(min_thickness 0.25)
+		(filled_areas_thickness no)
+		(fill yes
+			(thermal_gap 0.5)
+			(thermal_bridge_width 0.5)
+		)
+		(polygon
+			(pts
+				(xy 134.25 71.75) (xy 140 71.5) (xy 140 78.75) (xy 134.25 78.75)
+			)
+		)

Commit message: CNTRL v1.1 production
Routing:
- net PYRO_2: track 48.8 -> 46.7 mm
- net PYRO_1: track 52.9 -> 54.0 mm
- net GND: vias 55 -> 56
Changed lines of the file:
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@@
 	)
 	(via
-		(at 122.25 75.75)
+		(at 120.5 75.75)
 		(size 0.7)
 		(drill 0.3)
@@
 	)
 	(via
+		(at 125 66.25)
+		(size 0.7)
+		(drill 0.3)
+		(layers "F.Cu" "B.Cu")
+		(free yes)
+		(net 1)
+	)
+	(via
 		(at 115.5 82.75)
 		(size 0.7)
@@
 	)
 	(via
-		(at 139 78.25)
+		(at 139.5 78.25)
 		(size 0.7)
 		(drill 0.3)
@@
 	)
 	(via
-		(at 107.5 96.5)
+		(at 107.25 96.375)
 		(size 0.7)
 		(drill 0.3)
@@
 	)
 	(segment
-		(start 107.575 97.75)
-		(end 107.575 96.575)
+		(start 113.975 88.75)
+		(end 113.431634 88.206634)
 		(width 0.3)
 		(layer "B.Cu")
@@
 	(segment
 		(start 107.575 96.575)
-		(end 107.5 96.5)
-		(width 0.3)
-		(layer "B.Cu")
-		(net 5)
-	)
-	(segment
-		(start 113.975 88.75)
-		(end 113.431634 88.206634)
+		(end 107.575 97.75)
 		(width 0.3)
 		(layer "B.Cu")
@@
 	)
 	(segment
+		(start 107.375 96.375)
+		(end 107.575 96.575)
+		(width 0.3)
+		(layer "B.Cu")
+		(net 5)
+	)
+	(segment
 		(start 141.275 89.99)
 		(end 142.74 89.99)
@@
 	)
 	(segment
+		(start 107.25 96.375)
+		(end 107.375 96.375)
+		(width 0.3)
+		(layer "B.Cu")
+		(net 5)
+	)
+	(segment
 		(start 114.825 67.75)
 		(end 115.65 66.925)
@@
 	)
 	(segment
+		(start 94.75 109.5)
+		(end 94.25 109)
+		(width 0.5)
+		(layer "F.Cu")
+		(net 41)
+	)
+	(segment
+		(start 94.25 109)
+		(end 94.25 107.825)
+		(width 0.5)
+		(layer "F.Cu")
+		(net 41)
+	)
+	(segment
 		(start 94.25 107.825)
 		(end 92.425 106)
@@
 		(net 41)
 	)
-	(segment
-		(start 94.25 110)
-		(end 94.25 107.825)
-		(width 0.5)
-		(layer "F.Cu")
-		(net 41)
-	)
 	(via
-		(at 94.25 110)
+		(at 94.75 109.5)
 		(size 0.7)
 		(drill 0.3)
@@
 	)
 	(segment
-		(start 93.21967 111.03033)
-		(end 94.25 110)
+		(start 94.75 109.5)
+		(end 93.21967 111.03033)
 		(width 0.5)
 		(layer "B.Cu")
@@
 	)
 	(segment
-		(start 93.21967 111.033021)
-		(end 93.21967 111.03033)
+		(start 93.21967 111.03033)
+		(end 93.21967 111.033021)
 		(width 0.5)
 		(layer "B.Cu")
@@
 	)
 	(segment
-		(start 115.586668 84.85)
-		(end 107.15 84.85)
+		(start 91.625 108.508884)
+		(end 91.625 100.375)
 		(width 0.2)
 		(layer "In1.Cu")
@@
 	)
 	(segment
-		(start 116.736668 86)
-		(end 115.586668 84.85)
+		(start 93.116116 110)
+		(end 91.625 108.508884)
 		(width 0.2)
 		(layer "In1.Cu")
@@
 	)
 	(segment
-		(start 107.15 84.85)
-		(end 91.625 100.375)
+		(start 115.586668 84.85)
+		(end 116.736668 86)
 		(width 0.2)
 		(layer "In1.Cu")
@@
 	)
 	(segment
-		(start 118 86)
-		(end 116.736668 86)
+		(start 91.625 100.375)
+		(end 107.15 84.85)
 		(width 0.2)
 		(layer "In1.Cu")
@@
 	)
 	(segment
-		(start 93.116116 110)
-		(end 94.25 110)
+		(start 94.25 110)
+		(end 93.116116 110)
 		(width 0.2)
 		(layer "In1.Cu")
@@
 	)
 	(segment
-		(start 91.625 100.375)
-		(end 91.625 108.508884)
+		(start 107.15 84.85)
+		(end 115.586668 84.85)
 		(width 0.2)
 		(layer "In1.Cu")
@@
 	)
 	(segment
-		(start 91.625 108.508884)
-		(end 93.116116 110)
+		(start 116.736668 86)
+		(end 118 86)
+		(width 0.2)
+		(layer "In1.Cu")
+		(net 41)
+	)
+	(segment
+		(start 94.75 109.5)
+		(end 94.25 110)
 		(width 0.2)
 		(layer "In1.Cu")
@@
 	)
 	(segment
+		(start 100 112.75)
+		(end 99.925 112.75)
+		(width 0.5)
+		(layer "F.Cu")
+		(net 43)
+	)
+	(segment
 		(start 115.5 87)
 		(end 115.5 86.155202)
@@
 	)
 	(segment
-		(start 99.925 112.75)
+		(start 101 113.75)
 		(end 100 112.75)
 		(width 0.5)
@@
 	)
 	(segment
-		(start 101.5 116)
-		(end 100.5 116)
-		(width 0.5)
-		(layer "F.Cu")
-		(net 43)
-	)
-	(segment
-		(start 102 114.75)
-		(end 102 115.5)
-		(width 0.5)
-		(layer "F.Cu")
-		(net 43)
-	)
-	(segment
-		(start 100 112.75)
-		(end 102 114.75)
-		(width 0.5)
-		(layer "F.Cu")
-		(net 43)
-	)
-	(segment
-		(start 102 115.5)
-		(end 101.5 116)
+		(start 101 115.5)
+		(end 101 113.75)
 		(width 0.5)
 		(layer "F.Cu")
@@
 	)
 	(via
-		(at 100.5 116)
+		(at 101 115.5)
 		(size 0.7)
 		(drill 0.3)
@@
 	(segment
 		(start 99.46967 117.03033)
-		(end 100.5 116)
+		(end 99.46967 117.033021)
 		(width 0.5)
 		(layer "B.Cu")
@@
 	)
 	(segment
-		(start 99.46967 117.033021)
+		(start 101 115.5)
 		(end 99.46967 117.03033)
 		(width 0.5)
@@
 	)
 	(segment
-		(start 105.166186 90.8995)
-		(end 101.5 94.565686)
+		(start 101 115.5)
+		(end 101.5 115)
 		(width 0.2)
 		(layer "In1.Cu")
@@
 	)
 	(segment
-		(start 115.5 87)
-		(end 115.25 87.25)
+		(start 105.166186 90.8995)
+		(end 108.954349 90.8995)
 		(width 0.2)
 		(layer "In1.Cu")
@@
 	)
 	(segment
-		(start 101.5 115)
-		(end 100.5 116)
+		(start 101.5 94.565686)
+		(end 105.166186 90.8995)
 		(width 0.2)
 		(layer "In1.Cu")
@@
 	)
 	(segment
-		(start 115.25 87.25)
-		(end 112.603849 87.25)
+		(start 101.5 115)
+		(end 101.5 94.565686)
 		(width 0.2)
 		(layer "In1.Cu")
@@
 	(segment
 		(start 108.954349 90.8995)
-		(end 105.166186 90.8995)
+		(end 112.603849 87.25)
 		(width 0.2)
 		(layer "In1.Cu")
@@
 	)
 	(segment
-		(start 101.5 94.565686)
-		(end 101.5 115)
+		(start 115.25 87.25)
+		(end 115.5 87)
 		(width 0.2)
 		(layer "In1.Cu")
@@
 	(segment
 		(start 112.603849 87.25)
-		(end 108.954349 90.8995)
+		(end 115.25 87.25)
 		(width 0.2)
 		(layer "In1.Cu")
@@
 	)
 	(segment
-		(start 135.25 111.175)
-		(end 135.175 111.25)
-		(width 0.5)
-		(layer "F.Cu")
-		(net 57)
-	)
-	(segment
 		(start 115.5 91.5)
 		(end 114.5 90.5)
@@
 	)
 	(segment
-		(start 135.25 109.75)
-		(end 135.25 111.175)
+		(start 135.325 111.25)
+		(end 136.825 112.75)
 		(width 0.5)
 		(layer "F.Cu")
@@
 	)
 	(segment
-		(start 135.325 111.25)
-		(end 136.825 112.75)
+		(start 135.25 109.9)
+		(end 135.25 111.175)
 		(width 0.5)
 		(layer "F.Cu")
@@
 		(net 57)
 	)
+	(segment
+		(start 134.75 109.4)
+		(end 135.25 109.9)
+		(width 0.5)
+		(layer "F.Cu")
+		(net 57)
+	)
+	(segment
+		(start 135.25 111.175)
+		(end 135.175 111.25)
+		(width 0.5)
+		(layer "F.Cu")
+		(net 57)
+	)
 	(via
-		(at 135.25 109.75)
+		(at 134.75 109.4)
 		(size 0.7)
 		(drill 0.3)
@@
 	)
 	(segment
-		(start 111.4 93.15)
-		(end 111.4 91.781802)
+		(start 134.75 109.4)
+		(end 127.65 109.4)
 		(width 0.2)
 		(layer "In1.Cu")
@@
 	)
 	(segment
-		(start 111.4 91.781802)
-		(end 112.681802 90.5)
+		(start 114.5 90.5)
+		(end 115.5 91.5)
 		(width 0.2)
 		(layer "In1.Cu")
@@
 	)
 	(segment
-		(start 135.25 109.75)
-		(end 128 109.75)
+		(start 111.4 91.781802)
+		(end 112.681802 90.5)
 		(width 0.2)
 		(layer "In1.Cu")
@@
 	)
 	(segment
-		(start 128 109.75)
-		(end 111.4 93.15)
+		(start 111.4 93.15)
+		(end 111.4 91.781802)
 		(width 0.2)
 		(layer "In1.Cu")
@@
 	)
 	(segment
-		(start 114.5 90.5)
-		(end 115.5 91.5)
+		(start 127.65 109.4)
+		(end 111.4 93.15)
 		(width 0.2)
 		(layer "In1.Cu")
@@
 	)
 	(segment
-		(start 142.75 99.5)
-		(end 144.175 99.5)
-		(width 0.5)
-		(layer "B.Cu")
-		(net 58)
-	)
-	(segment
 		(start 145.825 101)
 		(end 145.675 101)
@@
 	)
 	(segment
-		(start 139.775215 96.025215)
-		(end 117.025215 96.025215)
-		(width 0.2)
-		(layer "In1.Cu")
+		(start 142.75 99.5)
+		(end 144.175 99.5)
+		(width 0.5)
+		(layer "B.Cu")
 		(net 58)
 	)
@@
 	)
 	(segment
-		(start 142.75 99.5)
-		(end 142.75 99)
+		(start 139.775215 96.025215)
+		(end 117.025215 96.025215)
 		(width 0.2)
 		(layer "In1.Cu")
@@
 		(width 0.2)
 		(layer "In1.Cu")
+		(net 58)
+	)
+	(segment
+		(start 142.75 99.5)
+		(end 142.75 99)
+		(width 0.2)
+		(layer "In1.Cu")
